File: first-pcb.kicad_pcb (KiCad board)
At the start: 2 copper layers, 0 parts

Commit message: Add Netlist
Netlist imported to PCB Editor and placed, along with making board shape.
Parts:
- added BT1: 9V, Battery:BatteryHolder_Eagle_12BH611-GR, F.Cu at (142.3, 102.5)
- added C1: 100nF, Capacitor_THT:C_Disc_D3.0mm_W2.0mm_P2.50mm, F.Cu at (163.4, 81.8)
- added K1: my_connector, Connector_PinHeader_2.54mm:PinHeader_1x02_P2.54mm_Vertical, F.Cu at (105.5, 114.6)
- added P1: 10k, Potentiometer_THT:Potentiometer_Alps_RK09K_Single_Vertical, F.Cu at (148.1, 84.7)
- added Q1: BC547, Package_TO_SOT_THT:TO-92_Inline, F.Cu at (91.8, 119.6)
- added R1: 100R, Resistor_THT:R_Axial_DIN0207_L6.3mm_D2.5mm_P10.16mm_Horizontal, F.Cu at (91.4, 114.3)
- added R2: 100R, Resistor_THT:R_Axial_DIN0207_L6.3mm_D2.5mm_P10.16mm_Horizontal, F.Cu at (148.0, 96.4)
- added U1: LM358, Package_DIP:DIP-8_W7.62mm, F.Cu at (148.0, 100.5)
Other:
- board outline added: 88.9 x 45.7 mm
