File: first-pcb.kicad_pcb (KiCad board)
At the start: 2 copper layers, 88.9 x 53.3 mm, 14 parts, among them K1 my_connector, P1 10k, Q1 BC547, U1 LM358

Commit message: Production Files
Parts:
- REF**: moved to B.Cu
- moved REF** 2.84 mm to (112.0, 95.5), turned to 180 degrees
